File: kicad/bd-tester/bd-tester.kicad_pcb (KiCad board)
At the start: 2 copper layers, 139.7 x 88.9 mm, 51 parts, among them J1 SM04B-SRSS, J2 PJ-202A, J3 MOLEX_9481054, J4 MOLEX_26605060, J5 Turret for DCC Phase A, J6 Turret for DCC Phase B, J7 AVR-ISP, SW1 FSM4JSMATR, U1 AP7381-50Y, U2 DRV8231A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

Commit message: DRC cleanup
Parts:
- moved R1 4.67 mm to (73.4, 46.5)
- moved R2 4.67 mm to (73.4, 43.9)
Routing:
- net Net-(U2-OUT2): track 39.9 -> 44.6 mm
- net Net-(D2-K): track 26.7 -> 31.4 mm
- net Net-(J6-Pin_1): track 187.6 -> 182.9 mm
- net Net-(J5-Pin_1): track 116.3 -> 111.7 mm
Changed lines of the file:
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@@
 	(footprint "Resistor_SMD:R_0805_2012Metric"
 		(layer "F.Cu")
-		(at 68.707 43.815 180)
+		(at 73.3806 43.8658 180)
 		(descr "Resistor SMD 0805 (2012 Metric), square (rectangular) end terminal, IPC-7351 nominal, (Body size source: IPC-SM-782 page 72, https://www.pcb-3d.com/wordpress/wp-content/uploads/ipc-sm-782a_amendment_1_and_2.pdf), generated with kicad-footprint-generator")
 		(tags "resistor")
@@
 	(footprint "Resistor_SMD:R_0805_2012Metric"
 		(layer "F.Cu")
-		(at 68.707 46.482 180)
+		(at 73.3806 46.5328 180)
 		(descr "Resistor SMD 0805 (2012 Metric), square (rectangular) end terminal, IPC-7351 nominal, (Body size source: IPC-SM-782 page 72, https://www.pcb-3d.com/wordpress/wp-content/uploads/ipc-sm-782a_amendment_1_and_2.pdf), generated with kicad-footprint-generator")
 		(tags "resistor")
@@
 	)
 	(gr_rect
-		(start 107.696 32.766)
-		(end 69.596 106.426)
+		(start 69.596 32.766)
+		(end 107.696 106.426)
 		(stroke
 			(width 0.15)
@@
 	)
 	(segment
-		(start 64.389 46.482)
-		(end 67.7945 46.482)
-		(width 1.016)
-		(layer "F.Cu")
-		(net 5)
-	)
-	(segment
-		(start 60.325 45.974)
-		(end 63.881 45.974)
-		(width 1.016)
-		(layer "F.Cu")
-		(net 5)
-	)
-	(segment
 		(start 56.007 48.768)
 		(end 56.007 48.006)
@@
 	)
 	(segment
+		(start 60.325 45.974)
+		(end 63.881 45.974)
+		(width 1.016)
+		(layer "F.Cu")
+		(net 5)
+	)
+	(segment
 		(start 56.007 51.054)
 		(end 56.007 48.768)
@@
 	)
 	(segment
-		(start 63.881 45.974)
-		(end 64.389 46.482)
+		(start 64.389 46.482)
+		(end 72.4173 46.482)
 		(width 1.016)
 		(layer "F.Cu")
@@
 	)
 	(segment
+		(start 63.881 45.974)
+		(end 64.389 46.482)
+		(width 1.016)
+		(layer "F.Cu")
+		(net 5)
+	)
+	(segment
 		(start 59.436 45.974)
 		(end 61.087 45.974)
@@
 		(net 5)
 	)
+	(segment
+		(start 72.4173 46.482)
+		(end 72.4681 46.5328)
+		(width 1.016)
+		(layer "F.Cu")
+		(net 5)
+	)
 	(via
 		(at 59.436 45.974)
@@
 	)
 	(segment
-		(start 129.032 43.815)
-		(end 131.191 41.656)
+		(start 74.2931 43.8658)
+		(end 128.9812 43.8658)
 		(width 1.016)
 		(layer "F.Cu")
@@
 	)
 	(segment
-		(start 153.162 32.766)
-		(end 153.162 39.751)
+		(start 128.9812 43.8658)
+		(end 131.191 41.656)
 		(width 1.016)
 		(layer "F.Cu")
@@
 	)
 	(segment
-		(start 153.162 39.751)
-		(end 155.633001 42.222001)
+		(start 153.061601 94.334399)
+		(end 151.257 96.139)
 		(width 1.016)
 		(layer "F.Cu")
@@
 	)
 	(segment
-		(start 153.061601 94.334399)
-		(end 151.257 96.139)
+		(start 153.162 32.766)
+		(end 153.162 39.751)
 		(width 1.016)
 		(layer "F.Cu")
@@
 	)
 	(segment
-		(start 155.633001 42.222001)
-		(end 157.170095 42.222001)
+		(start 153.162 39.751)
+		(end 155.633001 42.222001)
 		(width 1.016)
 		(layer "F.Cu")
@@
 	)
 	(segment
-		(start 69.6195 43.815)
-		(end 129.032 43.815)
+		(start 134.112 30.861)
+		(end 151.257 30.861)
 		(width 1.016)
 		(layer "F.Cu")
@@
 	)
 	(segment
-		(start 134.112 30.861)
-		(end 151.257 30.861)
+		(start 155.633001 42.222001)
+		(end 157.170095 42.222001)
 		(width 1.016)
 		(layer "F.Cu")
@@
 	)
 	(segment
+		(start 110.236 63.627)
+		(end 110.236 64.516)
+		(width 1.016)
+		(layer "F.Cu")
+		(net 28)
+	)
+	(segment
 		(start 106.68 46.482)
 		(end 110.236 50.038)
@@
 	)
 	(segment
-		(start 69.6195 46.482)
-		(end 106.68 46.482)
+		(start 110.236 64.516)
+		(end 110.236 65.405)
 		(width 1.016)
 		(layer "F.Cu")
@@
 	)
 	(segment
-		(start 110.236 63.627)
-		(end 110.236 64.516)
+		(start 127.957 106.045)
+		(end 129.689 107.777)
 		(width 1.016)
 		(layer "F.Cu")
@@
 	)
 	(segment
-		(start 110.236 64.516)
-		(end 110.236 65.405)
+		(start 110.236 50.038)
+		(end 110.236 63.627)
 		(width 1.016)
 		(layer "F.Cu")
@@
 	)
 	(segment
-		(start 127.957 106.045)
-		(end 129.689 107.777)
+		(start 74.2931 46.5328)
+		(end 74.3439 46.482)
 		(width 1.016)
 		(layer "F.Cu")
@@
 	)
 	(segment
-		(start 116.586 106.045)
-		(end 127.957 106.045)
+		(start 74.3439 46.482)
+		(end 106.68 46.482)
 		(width 1.016)
 		(layer "F.Cu")
@@
 	)
 	(segment
-		(start 110.236 50.038)
-		(end 110.236 63.627)
+		(start 116.586 106.045)
+		(end 127.957 106.045)
 		(width 1.016)
 		(layer "F.Cu")
@@
 	)
 	(segment
+		(start 64.389 43.815)
+		(end 63.754 44.45)
+		(width 1.016)
+		(layer "F.Cu")
+		(net 33)
+	)
+	(segment
 		(start 60.579 39.243)
 		(end 59.817 38.481)
@@
 	)
 	(segment
-		(start 63.754 44.45)
-		(end 60.579 44.45)
+		(start 72.4173 43.815)
+		(end 64.389 43.815)
 		(width 1.016)
 		(layer "F.Cu")
@@
 	)
 	(segment
-		(start 53.467 48.768)
-		(end 53.467 48.006)
+		(start 63.754 44.45)
+		(end 60.579 44.45)
 		(width 1.016)
 		(layer "F.Cu")
@@
 	)
 	(segment
-		(start 67.7945 43.815)
-		(end 64.389 43.815)
+		(start 53.467 48.768)
+		(end 53.467 48.006)
 		(width 1.016)
 		(layer "F.Cu")
@@
 	)
 	(segment
-		(start 64.389 43.815)
-		(end 63.754 44.45)
+		(start 72.4681 43.8658)
+		(end 72.4173 43.815)
 		(width 1.016)
 		(layer "F.Cu")
